File: electronics/v1/klara-circuitry.sch (KiCad schematic (older format))
At the start: 7 parts, among them IC1 ATtiny85

Commit message: evolution of schematic v1-v2-v3
Parts:
- C1, C2: value 1F -> 1.5F
- D1: value D_Zener -> Zener; Info (none) -> 5V
Other:
- moved on the sheet: C2
Changed lines of the file:
@@
 	1500 2600 1500 1750
 Wire Wire Line
-	3900 3450 3900 4300
-Wire Wire Line
-	3900 4300 2900 4300
-Wire Wire Line
-	1500 4300 1500 2900
+	3900 3450 3900 3850
 Wire Wire Line
 	1500 1750 1650 1750
@@
 P 2050 2750
 F 0 "D1" V 2004 2830 50  0000 L CNN
-F 1 "D_Zener" V 2095 2830 50  0000 L CNN
+F 1 "Zener" V 2095 2830 50  0000 L CNN
 F 2 "" H 2050 2750 50  0001 C CNN
 F 3 "~" H 2050 2750 50  0001 C CNN
+F 4 "5V" V 2188 2830 50  0000 L CNN "Info"
 	1    2050 2750
 	0    1    1    0
@@
 	2050 1750 2050 2600
 Wire Wire Line
-	2050 2900 2050 4300
-Connection ~ 2050 4300
+	2050 2900 2050 3850
 Wire Wire Line
-	2050 4300 1500 4300
+	2050 3850 1500 3850
 $Comp
 L Device:CP C1
@@
 P 2550 2750
 F 0 "C1" H 2668 2796 50  0000 L CNN
-F 1 "1F" H 2668 2705 50  0000 L CNN
+F 1 "1.5F" H 2668 2705 50  0000 L CNN
 F 2 "" H 2588 2600 50  0001 C CNN
 F 3 "~" H 2550 2750 50  0001 C CNN
@@
 L Device:CP C2
 U 1 1 62A6FA96
-P 2900 2750
-F 0 "C2" H 3018 2796 50  0000 L CNN
-F 1 "1F" H 3018 2705 50  0000 L CNN
-F 2 "" H 2938 2600 50  0001 C CNN
-F 3 "~" H 2900 2750 50  0001 C CNN
-	1    2900 2750
+P 3050 2750
+F 0 "C2" H 3168 2796 50  0000 L CNN
+F 1 "1.5F" H 3168 2705 50  0000 L CNN
+F 2 "" H 3088 2600 50  0001 C CNN
+F 3 "~" H 3050 2750 50  0001 C CNN
+	1    3050 2750
 	1    0    0    -1
 $EndComp
-Wire Wire Line
-	2050 1750 2550 1750
-Wire Wire Line
-	2550 1750 2550 2600
 Connection ~ 2050 1750
 Wire Wire Line
-	2550 1750 2900 1750
-Wire Wire Line
-	2900 1750 2900 2600
-Connection ~ 2550 1750
-Wire Wire Line
-	2550 2900 2550 4300
-Connection ~ 2550 4300
-Wire Wire Line
-	2550 4300 2050 4300
-Wire Wire Line
-	2900 2900 2900 4300
-Connection ~ 2900 4300
-Wire Wire Line
-	2900 4300 2550 4300
-Wire Wire Line
-	2900 1750 3900 1750
-Wire Wire Line
 	3900 1750 3900 2250
-Connection ~ 2900 1750
 Wire Wire Line
 	4700 2950 4700 2550
@@
 	5500 1750 5500 2250
 Connection ~ 3900 1750
-Wire Wire Line
-	5500 4300 5500 3050
-Connection ~ 3900 4300
 $Comp
 L Display_Character:HT1621 LCD1
@@
 	3900 1750 5500 1750
 Wire Wire Line
-	3900 4300 5500 4300
+	3900 3850 5500 3850
 Wire Wire Line
 	4700 2550 5100 2550
@@
 Wire Wire Line
 	4500 2950 4700 2950
+Connection ~ 3900 3850
+Wire Wire Line
+	5500 3850 5500 3050
+Connection ~ 2050 3850
+Wire Wire Line
+	1500 3850 1500 2900
+Wire Wire Line
+	2050 1750 2800 1750
+Wire Wire Line
+	2050 3850 2800 3850
+Wire Wire Line
+	2550 2600 2800 2600
+Wire Wire Line
+	2550 2900 2800 2900
+Wire Wire Line
+	2800 2600 2800 1750
+Connection ~ 2800 2600
+Wire Wire Line
+	2800 2600 3050 2600
+Connection ~ 2800 1750
+Wire Wire Line
+	2800 1750 3900 1750
+Wire Wire Line
+	2800 2900 2800 3850
+Connection ~ 2800 2900
+Wire Wire Line
+	2800 2900 3050 2900
+Connection ~ 2800 3850
+Wire Wire Line
+	2800 3850 3900 3850
 $EndSCHEMATC

Commit message: design & schematic wip
Parts:
- removed C2: 1.5F, symbol Device:CP
- renumbered D1 to D2, IC1 to U1
Other:
- moved on the sheet: C1
Changed lines of the file:
@@
 $EndDescr
 $Comp
-L MCU_Microchip_ATtiny:ATtiny85-20PU IC1
+L MCU_Microchip_ATtiny:ATtiny85-20PU U1
 U 1 1 62A64AD0
 P 3900 2850
-F 0 "IC1" H 3371 2896 50  0001 R CNN
+F 0 "U1" H 3703 3425 50  0000 R CNN
 F 1 "ATtiny85" H 4331 3425 50  0000 R CNN
 F 2 "Package_DIP:DIP-8_W7.62mm" H 3900 2850 50  0001 C CIN
@@
 	1500 1750 1650 1750
 $Comp
-L Device:D_Zener D1
+L Device:D_Zener D2
 U 1 1 62A6BF92
 P 2050 2750
-F 0 "D1" V 2004 2830 50  0000 L CNN
+F 0 "D2" V 2004 2830 50  0000 L CNN
 F 1 "Zener" V 2095 2830 50  0000 L CNN
 F 2 "" H 2050 2750 50  0001 C CNN
@@
 L Device:CP C1
 U 1 1 62A6F382
-P 2550 2750
-F 0 "C1" H 2668 2796 50  0000 L CNN
-F 1 "1.5F" H 2668 2705 50  0000 L CNN
-F 2 "" H 2588 2600 50  0001 C CNN
-F 3 "~" H 2550 2750 50  0001 C CNN
-	1    2550 2750
-	1    0    0    -1
-$EndComp
-$Comp
-L Device:CP C2
-U 1 1 62A6FA96
-P 3050 2750
-F 0 "C2" H 3168 2796 50  0000 L CNN
-F 1 "1.5F" H 3168 2705 50  0000 L CNN
-F 2 "" H 3088 2600 50  0001 C CNN
-F 3 "~" H 3050 2750 50  0001 C CNN
-	1    3050 2750
+P 2800 2750
+F 0 "C1" H 2918 2796 50  0000 L CNN
+F 1 "1.5F" H 2918 2705 50  0000 L CNN
+F 2 "" H 2838 2600 50  0001 C CNN
+F 3 "~" H 2800 2750 50  0001 C CNN
+	1    2800 2750
 	1    0    0    -1
 $EndComp
@@
 Wire Wire Line
 	2050 3850 2800 3850
-Wire Wire Line
-	2550 2600 2800 2600
-Wire Wire Line
-	2550 2900 2800 2900
-Wire Wire Line
-	2800 2600 2800 1750
-Connection ~ 2800 2600
-Wire Wire Line
-	2800 2600 3050 2600
 Connection ~ 2800 1750
 Wire Wire Line
@@
 Wire Wire Line
 	2800 2900 2800 3850
-Connection ~ 2800 2900
-Wire Wire Line
-	2800 2900 3050 2900
 Connection ~ 2800 3850
 Wire Wire Line
 	2800 3850 3900 3850
+Wire Wire Line
+	2800 1750 2800 2600
 $EndSCHEMATC
