File: electronics/v4/klara-circuitry.sch (KiCad schematic (older format))
At the start: 18 parts, among them SW1 Push, U1 MCP1700-3302E, U2 ATtiny85, U3 DS18B20

Commit message: PCB WIP
Parts:
- C1A, C1B: Field4 (none) -> 5.5V
- D2: Field5 (none) -> NZX5V1D.133; Info 5V -> 5.1V
Changed lines of the file:
@@
 F 2 "" H 2350 2750 50  0001 C CNN
 F 3 "~" H 2350 2750 50  0001 C CNN
-F 4 "5V" V 2488 2830 50  0000 L CNN "Info"
+F 4 "5.1V" V 2488 2830 50  0000 L CNN "Info"
+F 5 "NZX5V1D.133" V 2350 2750 50  0001 C CNN "Field5"
 	1    2350 2750
 	0    1    1    0
@@
 F 2 "" H 2838 2600 50  0001 C CNN
 F 3 "~" H 2800 2750 50  0001 C CNN
+F 4 "5.5V" H 2850 2550 50  0000 L CNN "Field4"
 	1    2800 2750
 	1    0    0    -1
@@
 F 2 "" H 3188 2600 50  0001 C CNN
 F 3 "~" H 3150 2750 50  0001 C CNN
+F 4 "5.5V" H 3200 2550 50  0000 L CNN "Field4"
 	1    3150 2750
 	1    0    0    -1
