File: electronics/v5/klara-circuitry.kicad_pcb (KiCad board)
At the start: 2 copper layers, 70 x 84 mm, 15 parts, among them J1 Pin header, U1 MCP1700-3302E, U3 ATtiny85

Commit message: design/pcb finalized for manufacturing
Parts:
- added G***: LOGO, Design:silk-text3, F.Cu at (134.6, 91.9)
- added G***: LOGO, Design:silk-text1, F.Cu at (101.3, 54.6)
- added G***: LOGO, Design:silk-text2, F.Cu at (110.5, 64.5)
- added G***: LOGO, design:stellar, F.Cu at (101.3, 46.7)
- C2: footprint Capacitor_THT:C_Rect_L4.0mm_W2.5mm_P2.50mm -> Capacitor_THT:C_Rect_L7.0mm_W2.0mm_P5.00mm
- moved C2 1.27 mm to (97.8, 91.4)
Routing:
- net Net-(C2-Pad1): track 72.8 -> 73.5 mm
- net Net-(C2-Pad2): track 193.1 -> 192.6 mm
Other:
- outline, holes or cut-outs redrawn
