File: electronics/v5/klara-circuitry.sch (KiCad schematic (older format))
At the start: 15 parts, among them J1 Pin header, U1 MCP1700-3302E, U3 ATtiny85

Commit message: design/pcb finalized for manufacturing
Parts:
- C2: footprint Capacitor_THT:C_Rect_L4.0mm_W2.5mm_P2.50mm -> Capacitor_THT:C_Rect_L7.0mm_W2.0mm_P5.00mm
- U1: footprint Package_TO_SOT_THT:TO-92_Inline -> Package_TO_SOT_THT:TO-92_Inline_Wide
Changed lines of the file:
@@
 F 0 "U1" H 3250 1850 50  0000 R CNN
 F 1 "MCP1700-3302E" H 3800 1600 50  0000 R CNN
-F 2 "Package_TO_SOT_THT:TO-92_Inline" H 3500 1550 50  0001 C CIN
+F 2 "Package_TO_SOT_THT:TO-92_Inline_Wide" H 3500 1550 50  0001 C CIN
 F 3 "http://ww1.microchip.com/downloads/en/DeviceDoc/20001826D.pdf" H 3500 1750 50  0001 C CNN
 	1    3500 1750
@@
 F 0 "C2" H 4065 1996 50  0000 L CNN
 F 1 "1uF" H 4065 1905 50  0000 L CNN
-F 2 "Capacitor_THT:C_Rect_L4.0mm_W2.5mm_P2.50mm" H 3988 1800 50  0001 C CNN
+F 2 "Capacitor_THT:C_Rect_L7.0mm_W2.0mm_P5.00mm" H 3988 1800 50  0001 C CNN
 F 3 "~" H 3950 1950 50  0001 C CNN
 	1    3950 1950
